File: Hardware/STAUB_BLIZZARD_107L/MowerBoard.kicad_pcb (KiCad board)
At the start: 4 copper layers, 54 x 120 mm, 103 parts, among them IC1 TPS62162DSGR, IC2 MC33978AES, IC3 PTPS274C65ASRHAR, IC4 TPS7B8601QDDARQ1, J1 432550083, J2 43045-0227, J3 39-28-1143, J4 SMA-J-P-H-ST-TH1, K1 V23086C2001A403, K2 V23086C2001A403, U1 AVR128DB48x-x6LX, U2 317990687

Commit message: Mise à jour du nom des pins dans le schématique et reprise du routage. Correction du PCB. Suppresion des SG inutilisés
Parts:
- removed C20, C21: 0.1uF, Capacitor_SMD:C_0402_1005Metric
- removed R12, R13: 100, Resistor_SMD:R_0603_1608Metric
- J1: footprint Lib:CONN_SDA_43255-00xx_06_MOL -> Custom:CONN_SDA_43255-00xx_06_MOL_NO_MARK
Connections:
- net /G_SP1 renamed /INPUT_BACKWARD
- net /G_SP2 renamed /OUT_AUX
- net /G_SP3 renamed /INPUT_FORWARD
- net /G_SP5 renamed /BT_AR
- net /G_SP6 renamed /INPUT_PTO_GS
- C18 pad 2: /G_SG0 -> /INPUT_SEAT
- C19 pad 2: /G_SG1 -> /INPUT_BRAKE
- C22 pad 2: /G_SP7 -> /INPUT_START
- C25 pad 2: /STARTER -> /PTO
- D18 pad 1: /STARTER -> /PTO
- D19 pad 1: /PTO -> /STARTER
- IC2 pad 7: Net-(IC2-SG2) -> unconnected-(IC2-SG2-Pad7)
- IC2 pad 8: Net-(IC2-SG3) -> unconnected-(IC2-SG3-Pad8)
- J1 pad 1: /PTO -> /STARTER
- J3 pad 10: /G_SP7 -> /INPUT_SEAT
- J3 pad 5: /STARTER -> /PTO
- J3 pad 8: /G_SG1 -> /INPUT_START
- J3 pad 9: /G_SG0 -> /INPUT_BRAKE
- K1 pad 14: /STARTER -> /PTO
- K1 pad 24: /PTO -> /STARTER
- R10 pad 1: /G_SG0 -> /INPUT_SEAT
- R11 pad 1: /G_SG1 -> /INPUT_BRAKE
- R14 pad 2: /G_SP7 -> /INPUT_START
- R17 pad 2: /STARTER -> /PTO
Routing:
- net /PTO: track 20.5 -> 78.4 mm
- net /STARTER: track 77.6 -> 20.5 mm
- net /INPUT_START: track 0.00 -> 14.6 mm, vias 0 -> 1
- net /INPUT_SEAT: track 0.00 -> 10.1 mm
- net /G_SG1: track 9.96 -> 0.00 mm
- net Net-(IC2-SG2): track 9.75 -> 0.00 mm
- net /INPUT_BRAKE: track 0.00 -> 9.44 mm
- net /G_SG0: track 9.30 -> 0.00 mm
- net /G_SP7: track 9.01 -> 0.00 mm
- net Net-(IC2-SG3): track 8.11 -> 0.00 mm
- net GND: track 31.0 -> 28.8 mm, vias 90 -> 106
- net /INPUT/SG3: track 1.69 -> 0.00 mm
- net /INPUT/SG2: track 1.69 -> 0.00 mm
- net (no net): vias 0 -> 6
