File: Hardware/STAUB_BLIZZARD_107L/MowerBoard.kicad_sch (KiCad schematic)
At the start: 11 parts, among them J1 432550083, J2 43045-0227, J3 39-28-1143

Commit message: Mise à jour du nom des pins dans le schématique et reprise du routage. Correction du PCB. Suppresion des SG inutilisés
Connections:
- net G_SG0 renamed INPUT_BRAKE
- net G_SG1 renamed INPUT_START
- net G_SP1 renamed INPUT_BACKWARD
- net G_SP2 renamed OUT_AUX
- net G_SP3 renamed INPUT_FORWARD
- net G_SP5 renamed BT_AR
- net G_SP6 renamed INPUT_PTO_GS
- net G_SP7 renamed INPUT_SEAT
- no-connect marks 8 -> 6
Other:
- sheet INPUT ports: added none; removed SG2, SG3
Changed lines of the file:
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@@
 	)
 	(no_connect
-		(at 132.08 107.95)
-	)
-	(no_connect
-		(at 132.08 105.41)
-	)
-	(no_connect
 		(at 138.43 38.1)
 	)
@@
 		)
 	)
-	(label "G_SP5"
+	(label "BT_AR"
 		(at 167.64 132.08 180)
 		(effects
@@
 		)
 	)
-	(label "G_SP3"
+	(label "INPUT_FORWARD"
 		(at 123.19 137.16 180)
 		(effects
@@
 		)
 	)
-	(label "G_SG0"
-		(at 123.19 127 180)
-		(effects
-			(font
-				(size 1.27 1.27)
-			)
-			(justify right bottom)
-		)
-	)
 	(label "STARTER"
 		(at 52.07 66.04 0)
@@
 		)
 	)
-	(label "G_SP2"
+	(label "OUT_AUX"
 		(at 82.55 55.88 180)
 		(effects
@@
 		)
 	)
-	(label "G_SP5"
+	(label "BT_AR"
 		(at 115.57 91.44 0)
 		(effects
@@
 		)
 	)
-	(label "G_SP7"
+	(label "INPUT_SEAT"
 		(at 123.19 129.54 180)
 		(effects
@@
 		)
 	)
-	(label "G_SP1"
-		(at 115.57 81.28 0)
+	(label "INPUT_PTO_GS"
+		(at 115.57 93.98 0)
 		(effects
 			(font
@@
 		)
 	)
-	(label "G_SG1"
-		(at 123.19 124.46 180)
+	(label "INPUT_FORWARD"
+		(at 115.57 86.36 0)
 		(effects
 			(font
 				(size 1.27 1.27)
 			)
-			(justify right bottom)
+			(justify left bottom)
 		)
 	)
-	(label "G_SP6"
-		(at 115.57 93.98 0)
+	(label "INPUT_BRAKE"
+		(at 123.19 127 180)
 		(effects
 			(font
 				(size 1.27 1.27)
 			)
-			(justify left bottom)
+			(justify right bottom)
 		)
 	)
-	(label "G_SP2"
-		(at 167.64 137.16 180)
+	(label "INPUT_BACKWARD"
+		(at 123.19 139.7 180)
 		(effects
 			(font
@@
 		)
 	)
-	(label "G_SG1"
-		(at 115.57 102.87 0)
+	(label "INPUT_BACKWARD"
+		(at 115.57 81.28 0)
 		(effects
 			(font
@@
 		)
 	)
-	(label "G_SP2"
-		(at 115.57 83.82 0)
+	(label "OUT_AUX"
+		(at 167.64 137.16 180)
 		(effects
 			(font
 				(size 1.27 1.27)
 			)
-			(justify left bottom)
+			(justify right bottom)
 		)
 	)
-	(label "G_SP1"
-		(at 123.19 139.7 180)
+	(label "INPUT_BRAKE"
+		(at 115.57 102.87 0)
 		(effects
 			(font
 				(size 1.27 1.27)
 			)
-			(justify right bottom)
+			(justify left bottom)
 		)
 	)
-	(label "G_SP7"
-		(at 115.57 96.52 0)
+	(label "OUT_AUX"
+		(at 115.57 83.82 0)
 		(effects
 			(font
@@
 		)
 	)
-	(label "VCC_FUSE10"
-		(at 82.55 41.91 0)
+	(label "INPUT_SEAT"
+		(at 115.57 100.33 0)
 		(effects
 			(font
@@
 		)
 	)
-	(label "G_SG0"
-		(at 115.57 100.33 0)
+	(label "VCC_FUSE10"
+		(at 82.55 41.91 0)
 		(effects
 			(font
@@
 		)
 	)
-	(label "G_SP6"
+	(label "INPUT_PTO_GS"
 		(at 167.64 129.54 180)
 		(effects
@@
 		)
 	)
+	(label "INPUT_START"
+		(at 123.19 124.46 180)
+		(effects
+			(font
+				(size 1.27 1.27)
+			)
+			(justify right bottom)
+		)
+	)
+	(label "INPUT_START"
+		(at 115.57 96.52 0)
+		(effects
+			(font
+				(size 1.27 1.27)
+			)
+			(justify left bottom)
+		)
+	)
 	(label "VCC_FUSE20"
 		(at 82.55 118.11 0)
@@
 		)
 	)
-	(label "G_SP3"
-		(at 115.57 86.36 0)
-		(effects
-			(font
-				(size 1.27 1.27)
-			)
-			(justify left bottom)
-		)
-	)
 	(symbol
 		(lib_id "Diode:SM6T6V8A")
@@
 			(effects
 				(font
-					(size 1.27 1.27)
-				)
-				(justify left)
-			)
-		)
-		(pin "SG2" input
-			(at 132.08 105.41 180)
-			(effects
-				(font
-					(size 1.27 1.27)
-				)
-				(justify left)
-			)
-		)
-		(pin "SG3" input
-			(at 132.08 107.95 180)
-			(effects
-				(font
